File: hardware/cirradio-devboard/cirradio-devboard.kicad_sch (KiCad schematic)
At the start: 0 parts

Commit message: add top-level schematic with hierarchical sheet references
Other:
- added sheet AD9361 + LVDS (ad9361.kicad_sch)
- added sheet Connectors & Debug (connectors.kicad_sch)
- added sheet DDR3L Memory (ddr3l.kicad_sch)
- added sheet Peripherals (peripherals.kicad_sch)
- added sheet Power Supply (power.kicad_sch)
- added sheet RF Front-End (rf-frontend.kicad_sch)
- added sheet Zynq-7045 (zynq.kicad_sch)
- note added: "+12V -> 5V/3.3V/1.8V/1.5V/1.35V/1.0V"
- note added: "+1V35, VTT"
- note added: "+1V8, +3V3A"
- note added: "+3V3"
- note added: "+3V3, +1V8"
- note added: "+3V3, +3V3A, +5V_PA"
- note added: "1. All inter-sheet signals use global labels - no explicit wires on top-level"
- note added: "2. Power sequencing: +5V -> +3V3/+3V3A -> +1V8 -> +1V5 -> +1V35 -> +1V0 -> PS_POR_B"
- note added: "225-512 MHz"
- note added: "2x MT41K256M16"
- note added: "3. DDR3L requires VTT termination and VTTREF midpoint from power sheet"
- note added: "4. AD9361 LVDS pairs: matched-length differential routing required"
- note added: "533 MHz / 1066 MT/s"
- note added: "AD9361 RF Transceiver"
- note added: "ARM Cortex-A9 + FPGA"
- note added: "CIRRADIO Tactical SDR - Top-Level Block Diagram"
- note added: "Connectors: PS_CLK, PS_UART0_TX/RX, PS_SPI_*, PS_I2C_*"
- note added: "DDR3 Bus (Addr/Data/Ctrl)"
- note added: "DDR3L x32 Memory"
- note added: "DESIGN NOTES"
- note added: "GPS, uSD, QSPI Flash"
- note added: "GbE, USB, I2C EEPROM"
- note added: "INTER-SHEET CONNECTIVITY (via Global Labels)"
- note added: "JTAG, UART, FMC-LPC"
- note added: "LNA, SAW, TX Driver, PA"
- note added: "LVDS Data + SPI Control"
- note added: "LVDS Data Interface"
- note added: "PL GPIO + JTAG/UART"
- note added: "PL GPIO Header"
- note added: "PS MIO + PL GPIO"
- note added: "PS MIO Groups"
- note added: "Peripherals: ETH_MDC, ETH_MDIO, GPS_1PPS"
- note added: "Power Management"
- note added: "Power Rails + POR"
- note added: "Power control: +1V0_EN/PG, +1V35_EN/PG, +1V5_EN/PG, +1V8_EN/PG, +3V3_EN/PG, +5V_EN/PG, PS_POR_B"
- note added: "Power rails: +1V0, +1V35, +1V5, +1V8, +3V3, +3V3A, +5V, +5V_PA, VTT, VTTREF"
- note added: "RF Ports (RX/TX)"
- note added: "SMA, BPF, T/R Switch"
- note added: "SPI Control"
- note added: "Sequenced rails, POR"
- note added: "Xilinx Zynq-7045 SoC"
Changed lines of the file:
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@@
     (comment 2 "Zynq-7045 + AD9361")
   )
+    (sheet (at 30 195) (size 60 30)
+      (stroke (width 0.001) (type solid))
+      (fill (color 255 255 255 1.0))
+      (property "Sheetname" "Power Supply" (at 30 194 0)
+        (effects (font (size 1.27 1.27))))
+      (property "Sheetfile" "power.kicad_sch" (at 30 226 0)
+        (effects (font (size 1.27 1.27))))
+    )
+    (sheet (at 145 105) (size 70 45)
+      (stroke (width 0.001) (type solid))
+      (fill (color 255 255 255 1.0))
+      (property "Sheetname" "Zynq-7045" (at 145 104 0)
+        (effects (font (size 1.27 1.27))))
+      (property "Sheetfile" "zynq.kicad_sch" (at 145 151 0)
+        (effects (font (size 1.27 1.27))))
+    )
+    (sheet (at 270 105) (size 55 35)
+      (stroke (width 0.001) (type solid))
+      (fill (color 255 255 255 1.0))
+      (property "Sheetname" "DDR3L Memory" (at 270 104 0)
+        (effects (font (size 1.27 1.27))))
+      (property "Sheetfile" "ddr3l.kicad_sch" (at 270 141 0)
+        (effects (font (size 1.27 1.27))))
+    )
+    (sheet (at 165 30) (size 65 40)
+      (stroke (width 0.001) (type solid))
+      (fill (color 255 255 255 1.0))
+      (property "Sheetname" "AD9361 + LVDS" (at 165 29 0)
+        (effects (font (size 1.27 1.27))))
+      (property "Sheetfile" "ad9361.kicad_sch" (at 165 71 0)
+        (effects (font (size 1.27 1.27))))
+    )
+    (sheet (at 30 30) (size 65 40)
+      (stroke (width 0.001) (type solid))
+      (fill (color 255 255 255 1.0))
+      (property "Sheetname" "RF Front-End" (at 30 29 0)
+        (effects (font (size 1.27 1.27))))
+      (property "Sheetfile" "rf-frontend.kicad_sch" (at 30 71 0)
+        (effects (font (size 1.27 1.27))))
+    )
+    (sheet (at 145 195) (size 65 30)
+      (stroke (width 0.001) (type solid))
+      (fill (color 255 255 255 1.0))
+      (property "Sheetname" "Peripherals" (at 145 194 0)
+        (effects (font (size 1.27 1.27))))
+      (property "Sheetfile" "peripherals.kicad_sch" (at 145 226 0)
+        (effects (font (size 1.27 1.27))))
+    )
+    (sheet (at 270 195) (size 65 30)
+      (stroke (width 0.001) (type solid))
+      (fill (color 255 255 255 1.0))
+      (property "Sheetname" "Connectors & Debug" (at 270 194 0)
+        (effects (font (size 1.27 1.27))))
+      (property "Sheetfile" "connectors.kicad_sch" (at 270 226 0)
+        (effects (font (size 1.27 1.27))))
+    )
+    (text "CIRRADIO Tactical SDR - Top-Level Block Diagram" (at 130 12 0) (effects (font (size 3.0 3.0))))
+    (text "225-512 MHz" (at 40 53 0) (effects (font (size 1.5 1.5))))
+    (text "SMA, BPF, T/R Switch" (at 40 57 0) (effects (font (size 1.27 1.27))))
+    (text "LNA, SAW, TX Driver, PA" (at 40 61 0) (effects (font (size 1.27 1.27))))
+    (text "AD9361 RF Transceiver" (at 175 43 0) (effects (font (size 1.5 1.5))))
+    (text "LVDS Data Interface" (at 175 47 0) (effects (font (size 1.27 1.27))))
+    (text "SPI Control" (at 175 51 0) (effects (font (size 1.27 1.27))))
+    (text "Xilinx Zynq-7045 SoC" (at 155 118 0) (effects (font (size 1.5 1.5))))
+    (text "ARM Cortex-A9 + FPGA" (at 155 122 0) (effects (font (size 1.27 1.27))))
+    (text "PS MIO + PL GPIO" (at 155 126 0) (effects (font (size 1.27 1.27))))
+    (text "DDR3L x32 Memory" (at 280 118 0) (effects (font (size 1.5 1.5))))
+    (text "2x MT41K256M16" (at 280 122 0) (effects (font (size 1.27 1.27))))
+    (text "533 MHz / 1066 MT/s" (at 280 126 0) (effects (font (size 1.27 1.27))))
+    (text "Power Management" (at 40 208 0) (effects (font (size 1.5 1.5))))
+    (text "+12V -> 5V/3.3V/1.8V/1.5V/1.35V/1.0V" (at 40 212 0) (effects (font (size 1.27 1.27))))
+    (text "Sequenced rails, POR" (at 40 216 0) (effects (font (size 1.27 1.27))))
+    (text "GbE, USB, I2C EEPROM" (at 155 208 0) (effects (font (size 1.5 1.5))))
+    (text "GPS, uSD, QSPI Flash" (at 155 212 0) (effects (font (size 1.27 1.27))))
+    (text "JTAG, UART, FMC-LPC" (at 280 208 0) (effects (font (size 1.5 1.5))))
+    (text "PL GPIO Header" (at 280 212 0) (effects (font (size 1.27 1.27))))
+    (polyline
+      (pts (xy 95 50) (xy 165 50))
+      (stroke (width 0.3) (type default) (color 0 100 0 1.0))
+    )
+    (text "RF Ports (RX/TX)" (at 110 46 0) (effects (font (size 1.27 1.27))))
+    (polyline
+      (pts (xy 195 70) (xy 180 105))
+      (stroke (width 0.3) (type default) (color 0 100 0 1.0))
+    )
+    (text "LVDS Data + SPI Control" (at 183 88 0) (effects (font (size 1.27 1.27))))
+    (polyline
+      (pts (xy 215 127) (xy 270 122))
+      (stroke (width 0.3) (type default) (color 0 100 0 1.0))
+    )
+    (text "DDR3 Bus (Addr/Data/Ctrl)" (at 225 115 0) (effects (font (size 1.27 1.27))))
+    (polyline
+      (pts (xy 180 150) (xy 180 195))
+      (stroke (width 0.3) (type default) (color 0 100 0 1.0))
+    )
+    (text "PS MIO Groups" (at 183 175 0) (effects (font (size 1.27 1.27))))
+    (polyline
+      (pts (xy 210 150) (xy 300 195))
+      (stroke (width 0.3) (type default) (color 0 100 0 1.0))
+    )
+    (text "PL GPIO + JTAG/UART" (at 240 170 0) (effects (font (size 1.27 1.27))))
+    (polyline
+      (pts (xy 60 195) (xy 60 155))
+      (stroke (width 0.3) (type default) (color 0 100 0 1.0))
+    )
+    (polyline
+      (pts (xy 60 155) (xy 145 135))
+      (stroke (width 0.3) (type default) (color 0 100 0 1.0))
+    )
+    (text "Power Rails + POR" (at 70 160 0) (effects (font (size 1.27 1.27))))
+    (polyline
+      (pts (xy 50 195) (xy 50 70))
+      (stroke (width 0.3) (type default) (color 0 100 0 1.0))
+    )
+    (text "+3V3, +3V3A, +5V_PA" (at 32 140 0) (effects (font (size 1.0 1.0))))
+    (polyline
+      (pts (xy 70 195) (xy 180 70))
+      (stroke (width 0.3) (type default) (color 0 100 0 1.0))
+    )
+    (text "+1V8, +3V3A" (at 110 130 0) (effects (font (size 1.0 1.0))))
+    (polyline
+      (pts (xy 80 195) (xy 290 140))
+      (stroke (width 0.3) (type default) (color 0 100 0 1.0))
+    )
+    (text "+1V35, VTT" (at 170 165 0) (effects (font (size 1.0 1.0))))
+    (polyline
+      (pts (xy 90 215) (xy 145 210))
+      (stroke (width 0.3) (type default) (color 0 100 0 1.0))
+    )
+    (text "+3V3, +1V8" (at 110 220 0) (effects (font (size 1.0 1.0))))
+    (polyline
+      (pts (xy 90 220) (xy 270 210))
+      (stroke (width 0.3) (type default) (color 0 100 0 1.0))
+    )
+    (text "+3V3" (at 175 222 0) (effects (font (size 1.0 1.0))))
+    (text "INTER-SHEET CONNECTIVITY (via Global Labels)" (at 30 250 0) (effects (font (size 2.0 2.0))))
+    (text "Power rails: +1V0, +1V35, +1V5, +1V8, +3V3, +3V3A, +5V, +5V_PA, VTT, VTTREF" (at 30 255 0) (effects (font (size 1.0 1.0))))
+    (text "Power control: +1V0_EN/PG, +1V35_EN/PG, +1V5_EN/PG, +1V8_EN/PG, +3V3_EN/PG, +5V_EN/PG, PS_POR_B" (at 30 259 0) (effects (font (size 1.0 1.0))))
+    (text "Peripherals: ETH_MDC, ETH_MDIO, GPS_1PPS" (at 30 263 0) (effects (font (size 1.0 1.0))))
+    (text "Connectors: PS_CLK, PS_UART0_TX/RX, PS_SPI_*, PS_I2C_*" (at 30 267 0) (effects (font (size 1.0 1.0))))
+    (text "DESIGN NOTES" (at 30 275 0) (effects (font (size 1.5 1.5))))
+    (text "1. All inter-sheet signals use global labels - no explicit wires on top-level" (at 30 279 0) (effects (font (size 1.0 1.0))))
+    (text "2. Power sequencing: +5V -> +3V3/+3V3A -> +1V8 -> +1V5 -> +1V35 -> +1V0 -> PS_POR_B" (at 30 283 0) (effects (font (size 1.0 1.0))))
+    (text "3. DDR3L requires VTT termination and VTTREF midpoint from power sheet" (at 30 287 0) (effects (font (size 1.0 1.0))))
+    (text "4. AD9361 LVDS pairs: matched-length differential routing required" (at 30 291 0) (effects (font (size 1.0 1.0))))
   (symbol_instances)
+  (sheet_instances
+    (path "/"
+      (page "1")
+    )
+  )
 )
